File: pcb/main/v101/3dsimo_kit.kicad_pcb (KiCad board)
At the start: 2 copper layers, 85 x 21 mm, 27 parts, among them J1 CONN_01X04, J2 CONN_01X04, J3 FiducialMark, J4 FiducialMark, J5 FiducialMark, J6 FiducialMark, M1 Motor, P1 PinHeader 2.54mm, Q1 IRLML0030, SW1 TACTM-64N-F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

Commit message: updated v101, added pcb and FW for KIT 2
Parts:
- turned Q1 to 180 degrees
